File: KiCad/GR_Loop_Switcher.sch (KiCad schematic (older format))
At the start: 69 parts, among them J1 Conn_01x02, J10 Conn_01x02, J11 Conn_01x02, J12 Conn_01x02, J13 Conn_01x02, J14 Conn_01x02, J15 Conn_01x02, J16 Conn_01x02, J17 Conn_01x02, J18 Conn_01x02, J19 Conn_01x02, J2 Conn_01x02, J20 Conn_01x02, J21 Conn_01x03, J22 Conn_01x02, J23 Conn_01x02, J24 Conn_01x02, J25 Conn_01x02, J26 Conn_01x02, J27 Conn_01x02, J28 Conn_01x02, J29 Conn_01x02, J3 Conn_01x02, J30 Conn_01x02, J31 Conn_01x02, J32 Conn_01x02, J33 Conn_01x02, J34 Conn_01x02, J35 Conn_01x02, J36 PJ-202A, J4 Conn_01x02, J5 Conn_01x02, J6 Conn_01x02, J7 Conn_01x02, J8 Conn_01x02, J9 Conn_01x02, Q1 2N7000, Q2 2N7000, U1 WeMos_D1_mini, U2 ICL7660, U3 MAX3485, U4 LM7805_TO220

Commit message: Add files via upload
Parts:
- C7: value 1uF -> 10uF
Changed lines of the file:
@@
 AR Path="/62B2822A" Ref="C7"  Part="1"
 F 0 "C7" H 2250 6375 50  0000 L CNN
-F 1 "1uF" H 2250 6275 50  0000 L CNN
+F 1 "10uF" H 2250 6275 50  0000 L CNN
 F 2 "Capacitor_THT:CP_Radial_D5.0mm_P2.50mm" H 2175 6325 50  0001 C CNN
 F 3 "~" H 2175 6325 50  0001 C CNN
